Commit message: little fixes

File: urdf/trash_robot.urdf.xacro (robot description, xacro)
@@ -1,245 +1,141 @@
 <?xml version="1.0"?>
+<!--
+  trash_robot.urdf.xacro — ЗЕРКАЛО only_robot.sdf
+  Имена ссылок, джоинтов и смещения взяты напрямую из SDF,
+  чтобы robot_state_publisher публиковал правильное TF-дерево.
+  Дерево:
+    base_link (= body в SDF, canonical_link)
+    ├── front_left_wheel   [revolute, front_left_wheel_joint]
+    ├── front_right_wheel  [revolute, front_right_wheel_joint]
+    ├── back_left_wheel    [revolute, back_left_wheel_joint]
+    ├── back_right_wheel   [revolute, back_right_wheel_joint]
+    ├── desk_for_depth     [fixed,    desk_for_depth_joint]
+    │   └── RGBD_camera    [fixed,    RGBD_camera_joint]
+    ├── nav_camera         [fixed,    nav_camera_joint]
+    └── lidar_link         [fixed,    lidar_joint]
+-->
 <robot xmlns:xacro="http://www.ros.org/wiki/xacro" name="trash_robot">
-  <!-- ==================== PROPERTIES ==================== -->
-  <xacro:property name="base_radius"   value="0.175"/>
-  <xacro:property name="base_height"   value="0.10"/>
-  <xacro:property name="base_mass"     value="5.0"/>
-  <xacro:property name="wheel_radius"  value="0.045"/>
-  <xacro:property name="wheel_width"   value="0.025"/>
-  <xacro:property name="wheel_mass"    value="0.3"/>
-  <xacro:property name="wheel_y_off"   value="0.19"/>
-  <xacro:property name="caster_radius" value="0.025"/>
-  <xacro:property name="caster_mass"   value="0.1"/>
-  <xacro:property name="lidar_size"    value="0.05"/>
-  <xacro:property name="lidar_mass"    value="0.2"/>
-  <xacro:property name="cam_x"    value="0.03"/>
-  <xacro:property name="cam_y"    value="0.015"/>
-  <xacro:property name="cam_z"    value="0.025"/>
-  <xacro:property name="cam_mass" value="0.05"/>
-  <!-- ==================== INERTIA MACROS ==================== -->
-  <xacro:macro name="cylinder_inertia" params="m r h">
-    <inertial>
-      <mass value="${m}"/>
-      <inertia ixx="${m*(3*r*r+h*h)/12}" ixy="0" ixz="0"
-               iyy="${m*(3*r*r+h*h)/12}" iyz="0"
-               izz="${m*r*r/2}"/>
-    </inertial>
-  </xacro:macro>
-  <xacro:macro name="box_inertia" params="m x y z">
-    <inertial>
-      <mass value="${m}"/>
-      <inertia ixx="${m*(y*y+z*z)/12}" ixy="0" ixz="0"
-               iyy="${m*(x*x+z*z)/12}" iyz="0"
-               izz="${m*(x*x+y*y)/12}"/>
-    </inertial>
-  </xacro:macro>
-  <xacro:macro name="sphere_inertia" params="m r">
-    <inertial>
-      <mass value="${m}"/>
-      <inertia ixx="${2*m*r*r/5}" ixy="0" ixz="0"
-               iyy="${2*m*r*r/5}" iyz="0"
-               izz="${2*m*r*r/5}"/>
-    </inertial>
-  </xacro:macro>
-  <!-- ==================== BASE ==================== -->
-  <link name="base_footprint"/>
-  <joint name="base_footprint_joint" type="fixed">
-    <parent link="base_footprint"/>
-    <child  link="base_link"/>
-    <origin xyz="0 0 ${wheel_radius}" rpy="0 0 0"/>
-  </joint>
+  <!-- ===== ТЕЛО (SDF body: 1.2×0.8×0.5м, масса 50кг) ===== -->
   <link name="base_link">
     <visual>
-      <geometry><cylinder radius="${base_radius}" length="${base_height}"/></geometry>
-      <material name="blue"><color rgba="0.2 0.4 0.8 1.0"/></material>
+      <geometry><box size="1.2 0.8 0.5"/></geometry>
+      <material name="blue"><color rgba="0.1 0.1 0.9 1.0"/></material>
     </visual>
     <collision>
-      <geometry><cylinder radius="${base_radius}" length="${base_height}"/></geometry>
+      <geometry><box size="1.2 0.8 0.5"/></geometry>
     </collision>
-    <xacro:cylinder_inertia m="${base_mass}" r="${base_radius}" h="${base_height}"/>
+    <inertial>
+      <mass value="50"/>
+      <inertia ixx="3.708333" ixy="0" ixz="0"
+               iyy="7.041667" iyz="0"
+               izz="8.666667"/>
+    </inertial>
   </link>
-  <!-- ==================== WHEEL MACRO ==================== -->
-  <xacro:macro name="wheel" params="name y_offset">
-    <link name="${name}_wheel_link">
+  <!-- ===== КОЛЁСА (SDF: radius=0.2, length=0.08) ===== -->
+  <!-- SDF pose relative_to body: (±0.40, ±0.44, -0.25), rpy=(-pi/2, 0, 0) -->
+  <xacro:macro name="wheel" params="name xyz_str">
+    <link name="${name}">
       <visual>
-        <origin xyz="0 0 0" rpy="${pi/2} 0 0"/>
-        <geometry><cylinder radius="${wheel_radius}" length="${wheel_width}"/></geometry>
-        <material name="black"><color rgba="0.1 0.1 0.1 1.0"/></material>
+        <origin rpy="1.5707963 0 0"/>
+        <geometry><cylinder radius="0.2" length="0.08"/></geometry>
+        <material name="darkgray"><color rgba="0.15 0.15 0.15 1"/></material>
       </visual>
       <collision>
-        <origin xyz="0 0 0" rpy="${pi/2} 0 0"/>
-        <geometry><cylinder radius="${wheel_radius}" length="${wheel_width}"/></geometry>
+        <origin rpy="1.5707963 0 0"/>
+        <geometry><cylinder radius="0.2" length="0.08"/></geometry>
       </collision>
-      <xacro:cylinder_inertia m="${wheel_mass}" r="${wheel_radius}" h="${wheel_width}"/>
+      <inertial>
+        <mass value="3"/>
+        <inertia ixx="0.0316" ixy="0" ixz="0"
+                 iyy="0.0316" iyz="0"
+                 izz="0.06"/>
+      </inertial>
     </link>
-    <joint name="${name}_wheel_joint" type="continuous">
+    <joint name="${name}_joint" type="continuous">
       <parent link="base_link"/>
-      <child  link="${name}_wheel_link"/>
-      <origin xyz="0 ${y_offset} 0" rpy="0 0 0"/>
+      <child  link="${name}"/>
+      <origin xyz="${xyz_str}" rpy="0 0 0"/>
       <axis xyz="0 1 0"/>
-      <dynamics damping="0.1" friction="0.1"/>
     </joint>
   </xacro:macro>
-  <xacro:wheel name="left"  y_offset=" ${wheel_y_off}"/>
-  <xacro:wheel name="right" y_offset="-${wheel_y_off}"/>
-  <!-- ==================== CASTERS ==================== -->
-  <xacro:macro name="caster" params="name x_offset">
-    <link name="${name}_caster_link">
-      <visual>
-        <geometry><sphere radius="${caster_radius}"/></geometry>
-        <material name="gray"><color rgba="0.5 0.5 0.5 1.0"/></material>
-      </visual>
-      <collision>
-        <geometry><sphere radius="${caster_radius}"/></geometry>
-      </collision>
-      <xacro:sphere_inertia m="${caster_mass}" r="${caster_radius}"/>
-    </link>
-    <joint name="${name}_caster_joint" type="fixed">
-      <parent link="base_link"/>
-      <child  link="${name}_caster_link"/>
-      <origin xyz="${x_offset} 0 ${-base_height/2 + caster_radius - wheel_radius}" rpy="0 0 0"/>
-    </joint>
-  </xacro:macro>
-  <xacro:caster name="front" x_offset=" ${base_radius - caster_radius}"/>
-  <xacro:caster name="rear"  x_offset="-${base_radius - caster_radius}"/>
-  <!-- ==================== LIDAR ==================== -->
+  <xacro:wheel name="front_left_wheel"  xyz_str=" 0.40  0.44 -0.25"/>
+  <xacro:wheel name="front_right_wheel" xyz_str=" 0.40 -0.44 -0.25"/>
+  <xacro:wheel name="back_left_wheel"   xyz_str="-0.40  0.44 -0.25"/>
+  <xacro:wheel name="back_right_wheel"  xyz_str="-0.40 -0.44 -0.25"/>
+  <!-- ===== СТОЙКА КАМЕРЫ (SDF desk_for_depth: 0.08×0.08×0.7м) ===== -->
+  <!-- pose relative_to body: (0.55, 0, 0.5) -->
+  <link name="desk_for_depth">
+    <visual>
+      <geometry><box size="0.08 0.08 0.7"/></geometry>
+      <material name="gray"><color rgba="0.3 0.3 0.3 1"/></material>
+    </visual>
+    <inertial>
+      <mass value="2.5"/>
+      <inertia ixx="0.1034" ixy="0" ixz="0"
+               iyy="0.1034" iyz="0"
+               izz="0.00267"/>
+    </inertial>
+  </link>
+  <joint name="desk_for_depth_joint" type="fixed">
+    <parent link="base_link"/>
+    <child  link="desk_for_depth"/>
+    <origin xyz="0.55 0 0.5" rpy="0 0 0"/>
+  </joint>
+  <!-- ===== RGBD-КАМЕРА (SDF: pose relative_to desk_for_depth) ===== -->
+  <!-- SDF: (0.05, 0, 0.33, 0, 0.872665, 0) — наклон вниз 50° -->
+  <link name="RGBD_camera">
+    <visual>
+      <geometry><box size="0.05 0.1 0.04"/></geometry>
+      <material name="black"><color rgba="0.05 0.05 0.05 1"/></material>
+    </visual>
+    <inertial>
+      <mass value="0.145"/>
+      <inertia ixx="0.0000604" ixy="0" ixz="0"
+               iyy="0.0000604" iyz="0"
+               izz="0.0000604"/>
+    </inertial>
+  </link>
+  <joint name="RGBD_camera_joint" type="fixed">
+    <parent link="desk_for_depth"/>
+    <child  link="RGBD_camera"/>
+    <!-- SDF pitch=0.872665 (наклон носом вниз) → в URDF rpy=(0, 0.872665, 0) -->
+    <origin xyz="0.05 0 0.33" rpy="0 0.872665 0"/>
+  </joint>
+  <!-- ===== НАВИГАЦИОННАЯ КАМЕРА (SDF: pose relative_to body) ===== -->
+  <!-- SDF: (0.6, 0, 0, 0, 0.0872665, 0) — небольшой наклон вниз 5° -->
+  <link name="nav_camera">
+    <visual>
+      <geometry><box size="0.05 0.1 0.04"/></geometry>
+      <material name="midgray"><color rgba="0.3 0.3 0.3 1"/></material>
+    </visual>
+    <inertial>
+      <mass value="0.145"/>
+      <inertia ixx="0.0000604" ixy="0" ixz="0"
+               iyy="0.0000604" iyz="0"
+               izz="0.0000604"/>
+    </inertial>
+  </link>
+  <joint name="nav_camera_joint" type="fixed">
+    <parent link="base_link"/>
+    <child  link="nav_camera"/>
+    <origin xyz="0.6 0 0" rpy="0 0.0872665 0"/>
+  </joint>
+  <!-- ===== ЛИДАР (SDF: pose relative_to body: 0 0 0.32) ===== -->
   <link name="lidar_link">
     <visual>
-      <geometry><cylinder radius="${lidar_size}" length="${lidar_size}"/></geometry>
-      <material name="black"><color rgba="0.1 0.1 0.1 1.0"/></material>
+      <geometry><cylinder radius="0.055" length="0.07"/></geometry>
+      <material name="lidar_black"><color rgba="0.1 0.1 0.1 1"/></material>
     </visual>
-    <collision>
-      <geometry><cylinder radius="${lidar_size}" length="${lidar_size}"/></geometry>
-    </collision>
-    <xacro:cylinder_inertia m="${lidar_mass}" r="${lidar_size}" h="${lidar_size}"/>
+    <inertial>
+      <mass value="0.2"/>
+      <inertia ixx="0.0002" ixy="0" ixz="0"
+               iyy="0.0002" iyz="0"
+               izz="0.0003"/>
+    </inertial>
   </link>
   <joint name="lidar_joint" type="fixed">
     <parent link="base_link"/>
     <child  link="lidar_link"/>
-    <origin xyz="0 0 ${base_height/2 + lidar_size/2}" rpy="0 0 0"/>
+    <origin xyz="0 0 0.32" rpy="0 0 0"/>
   </joint>
-  <!-- ==================== CAMERA ==================== -->
-  <link name="camera_link">
-    <visual>
-      <geometry><box size="${cam_x} ${cam_y} ${cam_z}"/></geometry>
-      <material name="red"><color rgba="0.8 0.1 0.1 1.0"/></material>
-    </visual>
-    <collision>
-      <geometry><box size="${cam_x} ${cam_y} ${cam_z}"/></geometry>
-    </collision>
-    <xacro:box_inertia m="${cam_mass}" x="${cam_x}" y="${cam_y}" z="${cam_z}"/>
-  </link>
-  <joint name="camera_joint" type="fixed">
-    <parent link="base_link"/>
-    <child  link="camera_link"/>
-    <origin xyz="${base_radius - 0.01} 0 ${base_height/4}" rpy="0 0 0"/>
-  </joint>
-  <!-- Optical frame (ROS convention: Z вперёд, X вправо, Y вниз) -->
-  <link name="camera_optical_link"/>
-  <joint name="camera_optical_joint" type="fixed">
-    <parent link="camera_link"/>
-    <child  link="camera_optical_link"/>
-    <origin xyz="0 0 0" rpy="${-pi/2} 0 ${-pi/2}"/>
-  </joint>
-  <!-- ==================== GAZEBO PLUGINS ==================== -->
-  <!-- Diff drive -->
-  <gazebo>
-    <plugin filename="gz-sim-diff-drive-system"
-            name="gz::sim::systems::DiffDrive">
-      <left_joint>left_wheel_joint</left_joint>
-      <right_joint>right_wheel_joint</right_joint>
-      <wheel_separation>${wheel_y_off * 2}</wheel_separation>
-      <wheel_radius>${wheel_radius}</wheel_radius>
-      <odom_publish_frequency>20</odom_publish_frequency>
-      <topic>/cmd_vel</topic>
-      <odom_topic>/odom</odom_topic>
-      <tf_topic>/tf</tf_topic>
-      <frame_id>odom</frame_id>
-      <child_frame_id>base_footprint</child_frame_id>
-      <max_linear_acceleration>1.0</max_linear_acceleration>
-    </plugin>
-  </gazebo>
-  <!-- Joint state publisher -->
-  <gazebo>
-    <plugin filename="gz-sim-joint-state-publisher-system"
-            name="gz::sim::systems::JointStatePublisher">
-      <topic>/joint_states</topic>
-    </plugin>
-  </gazebo>
-  <!-- Lidar (2D GPU ray) -->
-  <gazebo reference="lidar_link">
-    <sensor name="lidar" type="gpu_lidar">
-      <topic>/scan</topic>
-      <update_rate>10</update_rate>
-      <lidar>
-        <scan>
-          <horizontal>
-            <samples>360</samples>
-            <resolution>1</resolution>
-            <min_angle>-3.14159</min_angle>
-            <max_angle> 3.14159</max_angle>
-          </horizontal>
-        </scan>
-        <range>
-          <min>0.12</min>
-          <max>10.0</max>
-          <resolution>0.01</resolution>
-        </range>
-        <noise>
-          <type>gaussian</type>
-          <mean>0.0</mean>
-          <stddev>0.01</stddev>
-        </noise>
-      </lidar>
-      <always_on>true</always_on>
-      <visualize>true</visualize>
-    </sensor>
-  </gazebo>
-  <!-- RGB Camera -->
-  <gazebo reference="camera_link">
-    <sensor name="rgb_camera" type="camera">
-      <topic>/camera/image_raw</topic>
-      <camera_info_topic>/camera/camera_info</camera_info_topic>
-      <update_rate>30</update_rate>
-      <camera>
-        <horizontal_fov>1.047</horizontal_fov>
-        <image>
-          <width>640</width>
-          <height>480</height>
-          <format>R8G8B8</format>
-        </image>
-        <clip>
-          <near>0.1</near>
-          <far>100</far>
-        </clip>
-        <noise>
-          <type>gaussian</type>
-          <mean>0.0</mean>
-          <stddev>0.005</stddev>
-        </noise>
-      </camera>
-      <always_on>true</always_on>
-      <visualize>false</visualize>
-    </sensor>
-  </gazebo>
-  <!-- Колёса — трение для физики -->
-  <gazebo reference="left_wheel_link">
-    <mu1>1.0</mu1>
-    <mu2>1.0</mu2>
-    <kp>1e6</kp>
-    <kd>1.0</kd>
-  </gazebo>
-  <gazebo reference="right_wheel_link">
-    <mu1>1.0</mu1>
-    <mu2>1.0</mu2>
-    <kp>1e6</kp>
-    <kd>1.0</kd>
-  </gazebo>
-  <!-- Кастеры — скольжение -->
-  <gazebo reference="front_caster_link">
-    <mu1>0.01</mu1><mu2>0.01</mu2>
-  </gazebo>
-  <gazebo reference="rear_caster_link">
-    <mu1>0.01</mu1><mu2>0.01</mu2>
-  </gazebo>
 </robot>
