Commit message: Улучшения: реалистичные модели мусора, динамические препятствия, исправление карты
- worlds/trash_world.sdf: арена 26×26м (±13м), 25 реалистичных 3D-объектов
  (бутылки с горлышком/крышкой, банки на боку, коробки с клапанами, пакеты)
- scripts/navigator.py: файловый лог /tmp/trash_nav.log; динамические
  препятствия из лидара (scan_grid); MAP_HALF = 13.0; статус каждые 3с
- scripts/map_builder.py: MAP_HALF = 13.0; карта без серых «неизвестных» зон
- models/robot/only_robot.sdf + urdf/: углы камер скорректированы
  (RGBD 1.1 рад, nav 0.45 рад — лучший охват пола)
- tests/test_navigator.py: стены обновлены до ±13м (соответствие коду)
- README.md: обновлены размер арены и кол-во объектов

Co-Authored-By: Claude Sonnet 4.6 <noreply@anthropic.com>

File: urdf/trash_robot.urdf.xacro (robot description, xacro)
@@ -100,5 +100,5 @@
     <child  link="RGBD_camera"/>
     <!-- SDF pitch=0.872665 (наклон носом вниз) → в URDF rpy=(0, 0.872665, 0) -->
-    <origin xyz="0.05 0 0.33" rpy="0 0.872665 0"/>
+    <origin xyz="0.05 0 0.33" rpy="0 1.1 0"/>
   </joint>
   <!-- ===== НАВИГАЦИОННАЯ КАМЕРА (SDF: pose relative_to body) ===== -->
@@ -119,5 +119,5 @@
     <parent link="base_link"/>
     <child  link="nav_camera"/>
-    <origin xyz="0.6 0 0" rpy="0 0.0872665 0"/>
+    <origin xyz="0.6 0 0" rpy="0 0.45 0"/>
   </joint>
   <!-- ===== ЛИДАР (SDF: pose relative_to body: 0 0 0.32) ===== -->
